File: prototype/freerouting-addendum/freerouting-addendum.kicad_sch (KiCad schematic)
At the start: 25 parts, among them J2 battery, J3 5530843-5, J7 640456-3, J8 Micro_SD_Card, SW2 PWR_SWITCH, U1 RP2040, U11 TPS22919DCKR, U17 MODE_BTN, U18 SN74HCT373PWR, U2 BQ21040DBVR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

Commit message: finished calculator & mathboard PCBs, updated pricing calc
Parts:
- renumbered R2 to R6
